Commit message: added in friction

File: description/darm.urdf.xacro (robot description, xacro)
@@ -217,4 +217,5 @@
         <axis xyz="-2.3262389236353407e-63 -1.0 4.02455846426619e-16" />
         <limit lower="${-pi}" upper="${pi}" effort="20" velocity="2" />
+        <dynamics friction="0.2" />
     </joint>
     <joint name="joint_2_joint" type="revolute">
@@ -224,4 +225,5 @@
         <axis xyz="-3.730750440443123e-48 2.324793976983833e-16 1.0" />
         <limit lower="${-113 * pi / 180}" upper="${113 * pi / 180}" effort="40" velocity="2" />
+        <dynamics friction="0.2" />
     </joint>
     <joint name="joint_3_joint" type="revolute">
@@ -231,4 +233,5 @@
         <axis xyz="-2.3262389236353413e-63 -1.0 -4.413283944382435e-14" />
         <limit lower="${-pi}" upper="${pi}" effort="20" velocity="2" />
+        <dynamics friction="0.2" />
     </joint>
     <joint name="forearm_joint" type="revolute">
@@ -238,4 +241,5 @@
         <axis xyz="3.730750440443123e-48 -2.775557561585062e-17 1.0" />
         <limit lower="${-122.9 * pi / 180}" upper="${122.9 * pi / 180}" effort="20" velocity="2" />
+        <dynamics friction="0.2" />
     </joint>
     <joint name="differential_joint" type="revolute">
@@ -245,4 +249,5 @@
         <axis xyz="3.730750440443123e-48 6.683542608242411e-14 1.0" />
         <limit lower="${-110 * pi / 180}" upper="${110 * pi / 180}" effort="8" velocity="2" />
+        <dynamics friction="0.2" />
     </joint>
     <joint name="gripper_joint" type="revolute">
@@ -252,4 +257,5 @@
         <axis xyz="2.3262389236353413e-63 -1.0 -6.495339835895301e-14" />
         <limit lower="-3.141593" upper="3.141593" effort="8" velocity="2" />
+        <dynamics friction="0.2" />
     </joint>
     <joint name="finger_1_joint" type="prismatic">
@@ -259,4 +265,5 @@
         <axis xyz="-2.4967112710792502e-08 -1.4439660728622791e-53 0.9999999999999998" />
         <limit lower="-0.001" upper="0.025" effort="2" velocity="0.5" />
+        <dynamics friction="0.1" />
     </joint>
     <joint name="finger_2_joint" type="prismatic">
@@ -266,4 +273,5 @@
         <axis xyz="2.49671453513494e-08 1.262177448353619e-29 0.9999999999999997" />
         <limit lower="-0.001" upper="0.025" effort="2" velocity="0.5" />
+        <dynamics friction="0.1" />
     </joint>
     <joint name="dock_joint" type="fixed">
@@ -272,4 +280,5 @@
 		<child link="dock"/>
 	</joint>
+    <!-- Plugins -->
     <gazebo>
     <plugin

Commit message: Bake the initial 0 positions in to joint_2 and forearm_joint

File: description/darm.urdf.xacro (robot description, xacro)
@@ -221,5 +221,5 @@
     </joint>
     <joint name="joint_2_joint" type="revolute">
-        <origin xyz="-0.031000000000000003 -0.071 2.857436509628995e-17" rpy="-1.5707963267948963 -4.02455846426619e-16 -1.5707963267948966" />
+        <origin xyz="-0.031000000000000003 -0.071 2.857436509628995e-17" rpy="-1.5707963267948963 ${-113 * pi / 180} -1.5707963267948966" />" />
         <parent link="joint_1" />
         <child link="joint_2" />
@@ -237,5 +237,5 @@
     </joint>
     <joint name="forearm_joint" type="revolute">
-        <origin xyz="-0.0364 -0.065 -2.8686345638485836e-15" rpy="1.5707963267948966 4.413283944382435e-14 -1.5707963267948966" />
+        <origin xyz="-0.0364 -0.065 -2.8686345638485836e-15" rpy="1.5707963267948966 ${122.9 * pi / 180} -1.5707963267948966" />
         <parent link="joint_3" />
         <child link="forearm" />

Commit message: rotated robot by 180 degrees on Z axis, this puts the dock on the right side, which orients me when using the ps5 controller

File: description/darm.urdf.xacro (robot description, xacro)
@@ -208,5 +208,5 @@
     <!-- JOINTS -->
     <joint name="base_joint" type="fixed">
-        <origin xyz="0 0 0" rpy="${90 * pi / 180} 0 0"/>
+        <origin xyz="0 0 0" rpy="${90 * pi / 180} 0 ${180 * pi / 180}"/>
         <parent link="world"/>
         <child link="base_link"/>

Commit message: I should have opened a branch for this, this is a restore point because I'm about to re-export the URDF from fusion 360 with it 'pre-posed' in the dock, this should eliminate some rotation translation problems I'm having

File: description/darm.urdf.xacro (robot description, xacro)
@@ -225,5 +225,5 @@
         <child link="joint_2" />
         <axis xyz="-3.730750440443123e-48 2.324793976983833e-16 1.0" />
-        <limit lower="${-113 * pi / 180}" upper="${113 * pi / 180}" effort="40" velocity="2" />
+        <limit lower="-0.001" upper="${226 * pi / 180}" effort="40" velocity="2" />
         <dynamics friction="0.2" />
     </joint>
@@ -241,5 +241,5 @@
         <child link="forearm" />
         <axis xyz="3.730750440443123e-48 -2.775557561585062e-17 1.0" />
-        <limit lower="${-122.9 * pi / 180}" upper="${122.9 * pi / 180}" effort="20" velocity="2" />
+        <limit lower="-0.001" upper="${122.9 * pi / 180}" effort="20" velocity="2" />
         <dynamics friction="0.2" />
     </joint>
