Commit message: more cleanup

File: description/darm.urdf.xacro (robot description, xacro)
@@ -1,6 +1,8 @@
 <?xml version="1.0" ?>
 <robot name="darm_ros2" xmlns:xacro="http://www.ros.org/wiki/xacro">
+    <xacro:include filename="$(find darm_ros2)/description/darm.joints" />
+    <xacro:include filename="$(find darm_ros2)/description/darm.links" />
+    <xacro:include filename="$(find darm_ros2)/description/darm.trans" />
     <xacro:include filename="$(find darm_ros2)/description/materials.xacro" />
-    <xacro:include filename="$(find darm_ros2)/description/darm.trans" />
     <xacro:include filename="$(find darm_ros2)/description/ros2_control.xacro" />
     <!-- Gaebo Plugins -->
@@ -14,218 +16,3 @@
         </plugin>
     </gazebo>
-    <!-- Links -->
-	<link name="world" />
-    <link name="base_link">
-        <inertial>
-            <origin xyz="0 0 0.029745" rpy="0 0 0"/>
-            <mass value="3.946800"/>
-            <inertia ixx="0.043126" ixy="0" ixz="0" iyy="0.043126" iyz="0" izz="0.081135"/>
-        </inertial>
-        <visual>
-            <geometry> <mesh filename="package://darm_ros2/meshes/base_link.stl"/> </geometry>
-            <material name="orange"/>
-        </visual>
-        <collision>
-            <geometry> <mesh filename="package://darm_ros2/meshes/base_link.stl"/> </geometry>
-        </collision>
-    </link>
-    <link name="link_1">
-        <inertial>
-            <origin xyz="0 0 0.058438" rpy="0 0 0"/>
-            <mass value="0.929574"/>
-            <inertia ixx="0.002212" ixy="0" ixz="0" iyy="0.005558" iyz="0" izz="0.005049"/>
-        </inertial>
-        <visual>
-            <geometry> <mesh filename="package://darm_ros2/meshes/link_1.stl"/> </geometry>
-            <material name="orange"/>
-        </visual>
-        <collision>
-            <geometry> <mesh filename="package://darm_ros2/meshes/link_1.stl"/> </geometry>
-        </collision>
-    </link>
-    <link name="link_2">
-        <inertial>
-            <origin xyz="0 0 0.096970" rpy="0 0 0"/>
-            <mass value="0.599415"/>
-            <inertia ixx="0.002798" ixy="0" ixz="0" iyy="0.003048" iyz="0" izz="0.001145"/>
-        </inertial>
-        <visual>
-            <geometry> <mesh filename="package://darm_ros2/meshes/link_2.stl"/> </geometry>
-            <material name="orange"/>
-        </visual>
-        <collision>
-            <geometry> <mesh filename="package://darm_ros2/meshes/link_2.stl"/> </geometry>
-        </collision>
-    </link>
-    <link name="link_3">
-        <inertial>
-            <origin xyz="0.002679 0 0.056368" rpy="0 0 0"/>
-            <mass value="0.287967"/>
-            <inertia ixx="0.000711" ixy="0" ixz="-0.000002" iyy="0.000600" iyz="0" izz="0.000489"/>
-        </inertial>
-        <visual>
-            <geometry> <mesh filename="package://darm_ros2/meshes/link_3.stl"/> </geometry>
-            <material name="orange"/>
-        </visual>
-        <collision>
-            <geometry> <mesh filename="package://darm_ros2/meshes/link_3.stl"/> </geometry>
-        </collision>
-    </link>
-    <link name="forearm">
-        <inertial>
-            <origin xyz="-0.011120 0 0.139892" rpy="0 0 0"/>
-            <mass value="0.726179"/>
-            <inertia ixx="0.006041" ixy="0" ixz="-0.000871" iyy="0.007279" iyz="0" izz="0.001871"/>
-        </inertial>
-        <visual>
-            <geometry> <mesh filename="package://darm_ros2/meshes/forearm.stl"/> </geometry>
-            <material name="orange"/>
-        </visual>
-        <collision>
-            <geometry> <mesh filename="package://darm_ros2/meshes/forearm.stl"/> </geometry>
-        </collision>
-    </link>
-    <link name="differential">
-        <inertial>
-            <origin xyz="0 0 0.000544" rpy="0 0 0"/>
-            <mass value="0.124871"/>
-            <inertia ixx="0.000034" ixy="0" ixz="0" iyy="0.000147" iyz="0" izz="0.000145"/>
-        </inertial>
-        <visual>
-            <geometry> <mesh filename="package://darm_ros2/meshes/differential.stl"/> </geometry>
-            <material name="orange"/>
-        </visual>
-        <collision>
-            <geometry> <mesh filename="package://darm_ros2/meshes/differential.stl"/> </geometry>
-        </collision>
-    </link>
-    <link name="gripper">
-        <inertial>
-            <origin xyz="0 0 0.048627" rpy="0 0 0"/>
-            <mass value="0.227833"/>
-            <inertia ixx="0.000188" ixy="0" ixz="0" iyy="0.000227" iyz="0" izz="0.000181"/>
-        </inertial>
-        <visual>
-            <geometry> <mesh filename="package://darm_ros2/meshes/gripper.stl"/> </geometry>
-            <material name="orange"/>
-        </visual>
-        <collision>
-            <geometry> <mesh filename="package://darm_ros2/meshes/gripper.stl"/> </geometry>
-        </collision>
-    </link>
-    <link name="finger_1">
-        <inertial>
-            <origin xyz="-0.039715 0.004364 0.017475" rpy="0 0 0"/>
-            <mass value="0.033358"/>
-            <inertia ixx="0.000011" ixy="0" ixz="0" iyy="0.000012" iyz="0.000001" izz="0.000005"/>
-        </inertial>
-        <visual>
-            <geometry> <mesh filename="package://darm_ros2/meshes/finger_1.stl"/> </geometry>
-            <material name="rubber"/>
-        </visual>
-        <collision>
-            <geometry> <mesh filename="package://darm_ros2/meshes/finger_1.stl"/> </geometry>
-        </collision>
-    </link>
-    <link name="finger_2">
-        <inertial>
-            <origin xyz="0.039715 -0.004364 0.017475" rpy="0 0 0"/>
-            <mass value="0.033358"/>
-            <inertia ixx="0.000011" ixy="0" ixz="0" iyy="0.000012" iyz="-0.000001" izz="0.000005"/>
-        </inertial>
-        <visual>
-            <geometry> <mesh filename="package://darm_ros2/meshes/finger_2.stl"/> </geometry>
-            <material name="rubber"/>
-        </visual>
-        <collision>
-            <geometry> <mesh filename="package://darm_ros2/meshes/finger_2.stl"/> </geometry>
-        </collision>
-    </link>
-    <link name="dock">
-        <inertial>
-            <origin xyz="0 0.022445 -0.212158" rpy="0 0 0"/>
-            <mass value="0.527745"/>
-            <inertia ixx="0.000498" ixy="0" ixz="0" iyy="0.000998" iyz="0.000022" izz="0.000787"/>
-        </inertial>
-        <visual>
-            <geometry> <mesh filename="package://darm_ros2/meshes/dock.stl"/> </geometry>
-            <material name="rubber"/>
-        </visual>
-        <!-- No Collisions -->
-    </link>
-    <!-- Joints -->
-    <joint name="base_joint" type="fixed">
-        <origin xyz="0 0 0" rpy="0 0 0"/>
-        <parent link="world"/>
-        <child link="base_link"/>
-    </joint>
-    <joint name="link_1_joint" type="revolute">
-        <origin xyz="0 0 0.14444" rpy="0 0 0" />
-        <parent link="base_link" />
-        <child link="link_1" />
-        <axis xyz="0 0 1"/>
-        <limit lower="${-pi - 0.5}" upper="${pi + 0.5}" effort="5" velocity="10" />
-        <dynamics friction="0.2" />
-    </joint>
-    <joint name="link_2_joint" type="revolute">
-        <origin xyz="0 0 0.07556" rpy="${-113 * pi / 180} 0 0" />
-        <parent link="link_1" />
-        <child link="link_2" />
-        <axis xyz="1 0 0"/>
-        <limit lower="-0.001" upper="${226 * pi / 180}" effort="10" velocity="10" />
-        <dynamics friction="0.2" />
-    </joint>
-    <joint name="link_3_joint" type="revolute">
-        <origin xyz="0 0 0.18708" rpy="0 0 0" />
-        <parent link="link_2" />
-        <child link="link_3" />
-        <axis xyz="0 0 1" />
-        <limit lower="${-pi - 0.5}" upper="${pi + 0.5}" effort="5" velocity="10" />
-        <dynamics friction="0.2" />
-    </joint>
-    <joint name="forearm_joint" type="revolute">
-        <origin xyz="0 0 0.06292" rpy="${122.9 * pi / 180} 0 0" />
-        <parent link="link_3" />
-        <child link="forearm" />
-        <axis xyz="-1 0 0"/>
-        <limit lower="-0.001" upper="${245.8 * pi / 180}" effort="5" velocity="10" />
-        <dynamics friction="0.2" />
-    </joint>
-    <joint name="differential_joint" type="revolute">
-        <origin xyz="0 0 0.34" rpy="0 0 0" />
-        <parent link="forearm" />
-        <child link="differential" />
-        <axis xyz="1 0 0"/>
-        <limit lower="${-110 * pi / 180}" upper="${110 * pi / 180}" effort="2" velocity="10" />
-        <dynamics friction="0.2" />
-    </joint>
-    <joint name="gripper_joint" type="revolute">
-        <origin xyz="0 0 0.02" rpy="0 0 0" />
-        <parent link="differential" />
-        <child link="gripper" />
-        <axis xyz="0 0 -1" />
-        <limit lower="-3.141593" upper="3.141593" effort="2" velocity="10" />
-        <dynamics friction="0.2" />
-    </joint>
-    <joint name="finger_1_joint" type="prismatic">
-        <origin xyz="0.05 -0.0035 0.091365" rpy="0 0 0" />
-        <parent link="gripper" />
-        <child link="finger_1" />
-        <axis xyz="1 0 0"/>
-        <limit lower="-0.0001" upper="0.025" effort="1" velocity="2" />
-        <dynamics friction="0.2" />
-    </joint>
-    <joint name="finger_2_joint" type="prismatic">
-        <origin xyz="-0.05 0.0035 0.091365" rpy="0 0 0" />
-        <parent link="gripper" />
-        <child link="finger_2" />
-        <axis xyz="-1 0 0"/>
-        <limit lower="-0.0001" upper="0.025" effort="1" velocity="2" />
-        <dynamics friction="0.2" />
-    </joint>
-    <joint name="dock_joint" type="fixed">
-		<origin xyz="0 0 0" rpy="${90 * pi / 180} 0 0" />
-		<parent link="base_link"/>
-		<child link="dock"/>
-	</joint>
 </robot>

File: description/materials.xacro (robot description, xacro)
@@ -1,3 +1,4 @@
-<robot name="darm" xmlns:xacro="http://www.ros.org/wiki/xacro" >
+<?xml version="1.0"?>
+<robot xmlns:xacro="http://www.ros.org/wiki/xacro" >
     <material name="orange">
         <color rgba="1.0 0.329 0.0 1.0"/>
