Commit message: Should have opened a branch, some updates to the ros2_control.xacro

File: description/ros2_control.xacro (robot description, xacro)
@@ -2,7 +2,18 @@
 <robot xmlns:xacro="http://www.ros.org/wiki/xacro">
     <ros2_control name="darm_hardware" type="system">
-        <hardware>
-            <plugin>gz_ros2_control/GazeboSimSystem</plugin>
-        </hardware>
+        <!-- Select hardware type based on sim flag -->
+        <xacro:macro name="darm_ros2_control" params="sim:=false">
+            <if condition="${sim}">
+                    <hardware>
+                    <plugin>gz_ros2_control/GazeboSimSystem</plugin>
+                </hardware>
+            </if>
+            <unless condition="${sim}">
+                <hardware>
+                    <plugin>odrive_ros2_control_plugin/ODriveHardwareInterface</plugin>
+                    <param name="can">can0</param>
+                </hardware>
+            </unless>
+        </xacro:macro>
         <joint name="link_1_joint">
             <command_interface name="position"/>

Commit message: This is a working state, ugh

File: description/ros2_control.xacro (robot description, xacro)
@@ -2,18 +2,7 @@
 <robot xmlns:xacro="http://www.ros.org/wiki/xacro">
     <ros2_control name="darm_hardware" type="system">
-        <!-- Select hardware type based on sim flag -->
-        <xacro:macro name="darm_ros2_control" params="sim:=false">
-            <if condition="${sim}">
-                    <hardware>
-                    <plugin>gz_ros2_control/GazeboSimSystem</plugin>
-                </hardware>
-            </if>
-            <unless condition="${sim}">
-                <hardware>
-                    <plugin>odrive_ros2_control_plugin/ODriveHardwareInterface</plugin>
-                    <param name="can">can0</param>
-                </hardware>
-            </unless>
-        </xacro:macro>
+        <hardware>
+            <plugin>gz_ros2_control/GazeboSimSystem</plugin>
+        </hardware>
         <joint name="link_1_joint">
             <command_interface name="position"/>

Commit message: chagned ros2_control to look at the actuators defined in the .trans file, also added odrive node_ids, renamed actr to odrive for more clarity

File: description/ros2_control.xacro (robot description, xacro)
@@ -12,12 +12,36 @@
             </xacro:unless>
         </hardware>
-        <joint name="link_1_joint">         <command_interface name="position"/><state_interface name="velocity"/><state_interface name="position"/>    </joint>
-        <joint name="link_2_joint">         <command_interface name="position"/><state_interface name="velocity"/><state_interface name="position"/>    </joint>
-        <joint name="link_3_joint">         <command_interface name="position"/><state_interface name="velocity"/><state_interface name="position"/>    </joint>
-        <joint name="forearm_joint">        <command_interface name="position"/><state_interface name="velocity"/><state_interface name="position"/>    </joint>
-        <joint name="differential_joint">   <command_interface name="position"/><state_interface name="velocity"/><state_interface name="position"/>    </joint>
-        <joint name="gripper_joint">        <command_interface name="position"/><state_interface name="velocity"/><state_interface name="position"/>    </joint>
-        <joint name="finger_1_joint">       <command_interface name="position"/><state_interface name="velocity"/><state_interface name="position"/>    </joint>
-        <joint name="finger_2_joint">       <command_interface name="position"/><state_interface name="velocity"/><state_interface name="position"/>    </joint>
+    <joint name="joint_1_odrive">
+      <command_interface name="position"/><state_interface   name="position"/><state_interface   name="velocity"/>
+      <xacro:unless value="$(arg sim)"><param name="node_id">0</param></xacro:unless>
+    </joint>
+    <joint name="joint_2_left_odrive">
+      <command_interface name="position"/><state_interface   name="position"/><state_interface   name="velocity"/>
+      <xacro:unless value="$(arg sim)"><param name="node_id">1</param></xacro:unless>
+    </joint>
+    <joint name="joint_2_right_odrive">
+      <command_interface name="position"/><state_interface   name="position"/><state_interface   name="velocity"/>
+      <xacro:unless value="$(arg sim)"><param name="node_id">2</param></xacro:unless>
+    </joint>
+    <joint name="joint_3_odrive">
+      <command_interface name="position"/><state_interface   name="position"/><state_interface   name="velocity"/>
+      <xacro:unless value="$(arg sim)"><param name="node_id">3</param></xacro:unless>
+    </joint>
+    <joint name="forearm_odrive">
+      <command_interface name="position"/><state_interface   name="position"/><state_interface   name="velocity"/>
+      <xacro:unless value="$(arg sim)"><param name="node_id">4</param></xacro:unless>
+    </joint>
+    <joint name="diff_left_odrive">
+      <command_interface name="position"/><state_interface   name="position"/><state_interface   name="velocity"/>
+      <xacro:unless value="$(arg sim)"><param name="node_id">5</param></xacro:unless>
+    </joint>
+    <joint name="diff_right_odrive">
+      <command_interface name="position"/><state_interface   name="position"/><state_interface   name="velocity"/>
+      <xacro:unless value="$(arg sim)"><param name="node_id">6</param></xacro:unless>
+    </joint>
+    <joint name="finger_odrive">
+      <command_interface name="position"/><state_interface   name="position"/><state_interface   name="velocity"/>
+      <xacro:unless value="$(arg sim)"><param name="node_id">7</param></xacro:unless>
+    </joint>
     </ros2_control>
 </robot>

Commit message: ugh

File: description/ros2_control.xacro (robot description, xacro)
@@ -12,36 +12,12 @@
             </xacro:unless>
         </hardware>
-    <joint name="joint_1_odrive">
-      <command_interface name="position"/><state_interface   name="position"/><state_interface   name="velocity"/>
-      <xacro:unless value="$(arg sim)"><param name="node_id">0</param></xacro:unless>
-    </joint>
-    <joint name="joint_2_left_odrive">
-      <command_interface name="position"/><state_interface   name="position"/><state_interface   name="velocity"/>
-      <xacro:unless value="$(arg sim)"><param name="node_id">1</param></xacro:unless>
-    </joint>
-    <joint name="joint_2_right_odrive">
-      <command_interface name="position"/><state_interface   name="position"/><state_interface   name="velocity"/>
-      <xacro:unless value="$(arg sim)"><param name="node_id">2</param></xacro:unless>
-    </joint>
-    <joint name="joint_3_odrive">
-      <command_interface name="position"/><state_interface   name="position"/><state_interface   name="velocity"/>
-      <xacro:unless value="$(arg sim)"><param name="node_id">3</param></xacro:unless>
-    </joint>
-    <joint name="forearm_odrive">
-      <command_interface name="position"/><state_interface   name="position"/><state_interface   name="velocity"/>
-      <xacro:unless value="$(arg sim)"><param name="node_id">4</param></xacro:unless>
-    </joint>
-    <joint name="diff_left_odrive">
-      <command_interface name="position"/><state_interface   name="position"/><state_interface   name="velocity"/>
-      <xacro:unless value="$(arg sim)"><param name="node_id">5</param></xacro:unless>
-    </joint>
-    <joint name="diff_right_odrive">
-      <command_interface name="position"/><state_interface   name="position"/><state_interface   name="velocity"/>
-      <xacro:unless value="$(arg sim)"><param name="node_id">6</param></xacro:unless>
-    </joint>
-    <joint name="finger_odrive">
-      <command_interface name="position"/><state_interface   name="position"/><state_interface   name="velocity"/>
-      <xacro:unless value="$(arg sim)"><param name="node_id">7</param></xacro:unless>
-    </joint>
+        <joint name="link_1_joint">         <command_interface name="position"/><state_interface name="velocity"/><state_interface name="position"/>    </joint>
+        <joint name="link_2_joint">         <command_interface name="position"/><state_interface name="velocity"/><state_interface name="position"/>    </joint>
+        <joint name="link_3_joint">         <command_interface name="position"/><state_interface name="velocity"/><state_interface name="position"/>    </joint>
+        <joint name="forearm_joint">        <command_interface name="position"/><state_interface name="velocity"/><state_interface name="position"/>    </joint>
+        <joint name="differential_joint">   <command_interface name="position"/><state_interface name="velocity"/><state_interface name="position"/>    </joint>
+        <joint name="gripper_joint">        <command_interface name="position"/><state_interface name="velocity"/><state_interface name="position"/>    </joint>
+        <joint name="finger_1_joint">       <command_interface name="position"/><state_interface name="velocity"/><state_interface name="position"/>    </joint>
+        <joint name="finger_2_joint">       <command_interface name="position"/><state_interface name="velocity"/><state_interface name="position"/>    </joint>
     </ros2_control>
 </robot>

Commit message: testing crap

File: description/ros2_control.xacro (robot description, xacro)
@@ -1,23 +1,37 @@
 <?xml version="1.0"?>
 <robot xmlns:xacro="http://www.ros.org/wiki/xacro">
+  <!-- ===========================================================
+       1.  GAZEBO  (mechanical joints only, mock hardware)
+       =========================================================== -->
+  <xacro:if value="$(arg sim)">
+    <ros2_control name="darm_sim" type="system">
+      <hardware>
+        <plugin>gz_ros2_control/GazeboSimSystem</plugin>
+      </hardware>
+      <joint name="link_1_joint">       <command_interface name="position"/> <state_interface name="position"/> <state_interface name="velocity"/></joint>
+      <joint name="link_2_joint">       <command_interface name="position"/> <state_interface name="position"/> <state_interface name="velocity"/></joint>
+      <joint name="link_3_joint">       <command_interface name="position"/> <state_interface name="position"/> <state_interface name="velocity"/></joint>
+      <joint name="forearm_joint">      <command_interface name="position"/> <state_interface name="position"/> <state_interface name="velocity"/></joint>
+      <joint name="differential_joint"> <command_interface name="position"/> <state_interface name="position"/> <state_interface name="velocity"/></joint>
+      <joint name="gripper_joint">      <command_interface name="position"/> <state_interface name="position"/> <state_interface name="velocity"/></joint>
+      <joint name="finger_1_joint">     <command_interface name="position"/> <state_interface name="position"/> <state_interface name="velocity"/></joint>
+      <joint name="finger_2_joint">     <command_interface name="position"/> <state_interface name="position"/> <state_interface name="velocity"/></joint>
+    </ros2_control>
+  </xacro:if>
+  <xacro:unless value="$(arg sim)">
     <ros2_control name="darm_hardware" type="system">
-        <!-- Select GZ Sim or Odrive hardware interface based on 'sim' -->
-        <hardware>
-            <xacro:if value="$(arg sim)">
-                <plugin>gz_ros2_control/GazeboSimSystem</plugin>
-            </xacro:if>
-            <xacro:unless value="$(arg sim)">
-                <plugin>odrive_ros2_control_plugin/ODriveHardwareInterface</plugin>
-                <param name="can">can0</param>
-            </xacro:unless>
-        </hardware>
-        <joint name="link_1_joint">         <command_interface name="position"/><state_interface name="velocity"/><state_interface name="position"/>    </joint>
-        <joint name="link_2_joint">         <command_interface name="position"/><state_interface name="velocity"/><state_interface name="position"/>    </joint>
-        <joint name="link_3_joint">         <command_interface name="position"/><state_interface name="velocity"/><state_interface name="position"/>    </joint>
-        <joint name="forearm_joint">        <command_interface name="position"/><state_interface name="velocity"/><state_interface name="position"/>    </joint>
-        <joint name="differential_joint">   <command_interface name="position"/><state_interface name="velocity"/><state_interface name="position"/>    </joint>
-        <joint name="gripper_joint">        <command_interface name="position"/><state_interface name="velocity"/><state_interface name="position"/>    </joint>
-        <joint name="finger_1_joint">       <command_interface name="position"/><state_interface name="velocity"/><state_interface name="position"/>    </joint>
-        <joint name="finger_2_joint">       <command_interface name="position"/><state_interface name="velocity"/><state_interface name="position"/>    </joint>
+      <hardware>
+        <plugin>odrive_ros2_control_plugin/ODriveHardwareInterface</plugin>
+        <param name="can">can0</param>
+      </hardware>
+      <joint name="joint_1_actr">       <command_interface name="position"/> <state_interface name="position"/> <state_interface name="velocity"/> <param name="node_id">1</param></joint>
+      <joint name="joint_2_left_actr">  <command_interface name="position"/> <state_interface name="position"/> <state_interface name="velocity"/> <param name="node_id">2</param></joint>
+      <joint name="joint_2_right_actr"> <command_interface name="position"/> <state_interface name="position"/> <state_interface name="velocity"/> <param name="node_id">3</param></joint>
+      <joint name="joint_3_actr">       <command_interface name="position"/> <state_interface name="position"/> <state_interface name="velocity"/> <param name="node_id">4</param></joint>
+      <joint name="forearm_actr">       <command_interface name="position"/> <state_interface name="position"/> <state_interface name="velocity"/> <param name="node_id">5</param></joint>
+      <joint name="diff_left_actr">     <command_interface name="position"/> <state_interface name="position"/> <state_interface name="velocity"/> <param name="node_id">6</param></joint>
+      <joint name="diff_right_actr">    <command_interface name="position"/> <state_interface name="position"/> <state_interface name="velocity"/> <param name="node_id">7</param></joint>
+      <joint name="finger_actr">        <command_interface name="position"/> <state_interface name="position"/> <state_interface name="velocity"/> <param name="node_id">8</param></joint>
     </ros2_control>
+  </xacro:unless>
 </robot>

Commit message: revereted ros2 control file.....

File: description/ros2_control.xacro (robot description, xacro)
@@ -1,37 +1,23 @@
 <?xml version="1.0"?>
 <robot xmlns:xacro="http://www.ros.org/wiki/xacro">
-  <!-- ===========================================================
-       1.  GAZEBO  (mechanical joints only, mock hardware)
-       =========================================================== -->
-  <xacro:if value="$(arg sim)">
-    <ros2_control name="darm_sim" type="system">
-      <hardware>
-        <plugin>gz_ros2_control/GazeboSimSystem</plugin>
-      </hardware>
-      <joint name="link_1_joint">       <command_interface name="position"/> <state_interface name="position"/> <state_interface name="velocity"/></joint>
-      <joint name="link_2_joint">       <command_interface name="position"/> <state_interface name="position"/> <state_interface name="velocity"/></joint>
-      <joint name="link_3_joint">       <command_interface name="position"/> <state_interface name="position"/> <state_interface name="velocity"/></joint>
-      <joint name="forearm_joint">      <command_interface name="position"/> <state_interface name="position"/> <state_interface name="velocity"/></joint>
-      <joint name="differential_joint"> <command_interface name="position"/> <state_interface name="position"/> <state_interface name="velocity"/></joint>
-      <joint name="gripper_joint">      <command_interface name="position"/> <state_interface name="position"/> <state_interface name="velocity"/></joint>
-      <joint name="finger_1_joint">     <command_interface name="position"/> <state_interface name="position"/> <state_interface name="velocity"/></joint>
-      <joint name="finger_2_joint">     <command_interface name="position"/> <state_interface name="position"/> <state_interface name="velocity"/></joint>
+    <ros2_control name="darm_hardware" type="system">
+        <!-- Select GZ Sim or Odrive hardware interface based on 'sim' -->
+        <hardware>
+            <xacro:if value="$(arg sim)">
+                <plugin>gz_ros2_control/GazeboSimSystem</plugin>
+            </xacro:if>
+            <xacro:unless value="$(arg sim)">
+                <plugin>odrive_ros2_control_plugin/ODriveHardwareInterface</plugin>
+                <param name="can">can0</param>
+            </xacro:unless>
+        </hardware>
+        <joint name="link_1_joint">         <command_interface name="position"/><state_interface name="velocity"/><state_interface name="position"/>    </joint>
+        <joint name="link_2_joint">         <command_interface name="position"/><state_interface name="velocity"/><state_interface name="position"/>    </joint>
+        <joint name="link_3_joint">         <command_interface name="position"/><state_interface name="velocity"/><state_interface name="position"/>    </joint>
+        <joint name="forearm_joint">        <command_interface name="position"/><state_interface name="velocity"/><state_interface name="position"/>    </joint>
+        <joint name="differential_joint">   <command_interface name="position"/><state_interface name="velocity"/><state_interface name="position"/>    </joint>
+        <joint name="gripper_joint">        <command_interface name="position"/><state_interface name="velocity"/><state_interface name="position"/>    </joint>
+        <joint name="finger_1_joint">       <command_interface name="position"/><state_interface name="velocity"/><state_interface name="position"/>    </joint>
+        <joint name="finger_2_joint">       <command_interface name="position"/><state_interface name="velocity"/><state_interface name="position"/>    </joint>
     </ros2_control>
-  </xacro:if>
-  <xacro:unless value="$(arg sim)">
-    <ros2_control name="darm_hardware" type="system">
-      <hardware>
-        <plugin>odrive_ros2_control_plugin/ODriveHardwareInterface</plugin>
-        <param name="can">can0</param>
-      </hardware>
-      <joint name="joint_1_actr">       <command_interface name="position"/> <state_interface name="position"/> <state_interface name="velocity"/> <param name="node_id">1</param></joint>
-      <joint name="joint_2_left_actr">  <command_interface name="position"/> <state_interface name="position"/> <state_interface name="velocity"/> <param name="node_id">2</param></joint>
-      <joint name="joint_2_right_actr"> <command_interface name="position"/> <state_interface name="position"/> <state_interface name="velocity"/> <param name="node_id">3</param></joint>
-      <joint name="joint_3_actr">       <command_interface name="position"/> <state_interface name="position"/> <state_interface name="velocity"/> <param name="node_id">4</param></joint>
-      <joint name="forearm_actr">       <command_interface name="position"/> <state_interface name="position"/> <state_interface name="velocity"/> <param name="node_id">5</param></joint>
-      <joint name="diff_left_actr">     <command_interface name="position"/> <state_interface name="position"/> <state_interface name="velocity"/> <param name="node_id">6</param></joint>
-      <joint name="diff_right_actr">    <command_interface name="position"/> <state_interface name="position"/> <state_interface name="velocity"/> <param name="node_id">7</param></joint>
-      <joint name="finger_actr">        <command_interface name="position"/> <state_interface name="position"/> <state_interface name="velocity"/> <param name="node_id">8</param></joint>
-    </ros2_control>
-  </xacro:unless>
 </robot>
